File: SPI-Gyro-shield/Hardware/Arduino_kuukulgur-alternatiivne.brd (EAGLE design)
At the start: 101.6 x 53.3 mm, 162 parts, among them IC2 TPS77333DGK, T1 BD651, U1 MPU-6000QFN-24, U2 txb0108, Y1 CSTCE16M0V53-R0 16MHZ

Commit message: Minor bugfixes to boards.
Parts:
- Y1: value CSTCE16M0V53-R0 16MHZ -> CSTCE8M00G15C99-R0
- moved R44 27.5 mm to (15.8, 20.3), turned to 180 degrees
Changed lines of the file:
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@@
 <element name="JP17" library="pinhead" package="1X09" value="" x="65.9" y="34.8" rot="R270"/>
 <element name="JP18" library="pinhead" package="1X09" value="" x="60.7" y="34.8" rot="R270"/>
-<element name="Y1" library="SmartPrj" package="RESONATOR" value="CSTCE16M0V53-R0 16MHZ" x="26.7983" y="20.9662"/>
+<element name="Y1" library="SmartPrj" package="RESONATOR" value="CSTCE8M00G15C99-R0" x="26.7983" y="20.9662"/>
 <element name="C1" library="SmartPrj" package="C0603-ROUND" value="100n" x="15.1915" y="29.5848" rot="R180"/>
 <element name="C5" library="SmartPrj" package="C0603-ROUND" value="100n" x="15.1883" y="27.5476" rot="R180"/>
@@
 <element name="C30" library="rcl" package="C/6032-28R" value="47uF/16V" x="2.8" y="12.5" rot="R90"/>
 <element name="C31" library="rcl" package="C/6032-28R" value="47uF/10V" x="90.7" y="48.3" rot="R90"/>
-<element name="R44" library="SmartPrj" package="R0603-ROUND" value="47k" x="0.8" y="-2.7"/>
+<element name="R44" library="SmartPrj" package="R0603-ROUND" value="47k" x="15.8" y="20.3" rot="R180"/>
 </elements>
 <signals>
@@
 <wire x1="14.2993" y1="29.5816" x2="14.3025" y2="29.5848" width="1.016" layer="1"/>
 <contactref element="R44" pad="2"/>
-<wire x1="1.689" y1="-2.7" x2="2.8369" y2="4.0752" width="0" layer="19" extent="1-1"/>
+<wire x1="11.45" y1="20.0048" x2="14.911" y2="20.3" width="0" layer="19" extent="1-16"/>
 </signal>
 <signal name="+3V3" class="1">
@@
 <contactref element="R44" pad="1"/>
 <contactref element="MCU" pad="4"/>
-<wire x1="-0.089" y1="-2.7" x2="22.2" y2="25" width="0" layer="19" extent="1-1"/>
+<wire x1="16.689" y1="20.3" x2="22.2" y2="25" width="0" layer="19" extent="1-1"/>
 </signal>
 </signals>

Commit message: Clarifications in schematic
Connections:
- net CS2_3V renamed CS_MOTOR_3V
- net CS_3V renamed CS_GYRO_3V
- net INT2_3V renamed RESET_MOTOR_3V
- net INT_3V renamed INT_GYRO_3V
Changed lines of the file:
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@@
 <via x="30.4039" y="44.0114" extent="1-16" drill="0.4064" diameter="0.9144"/>
 </signal>
-<signal name="INT_3V">
+<signal name="INT_GYRO_3V">
 <contactref element="U1" pad="12"/>
 <contactref element="U2" pad="5"/>
@@
 <via x="77.3413" y="20.8393" extent="1-16" drill="0.4064" diameter="0.9144"/>
 </signal>
-<signal name="CS_3V">
+<signal name="CS_GYRO_3V">
 <contactref element="U1" pad="8"/>
 <contactref element="U2" pad="1"/>
@@
 <wire x1="46.648" y1="32.337" x2="48.211" y2="33.9" width="0.2032" layer="1"/>
 </signal>
-<signal name="CS2_3V">
+<signal name="CS_MOTOR_3V">
 <contactref element="U2" pad="8"/>
 <contactref element="MCU" pad="16"/>
@@
 <via x="29.2014" y="5.8742" extent="1-16" drill="0.4064" diameter="0.9144"/>
 </signal>
-<signal name="INT2_3V">
+<signal name="RESET_MOTOR_3V">
 <contactref element="U2" pad="9"/>
 <contactref element="MCU" pad="18"/>
