File: SPI-Gyro-shield/Hardware/Arduino_kuukulgur-alternatiivne.sch (EAGLE design)
At the start: 162 parts, among them IC2 TPS77333DGK, T1 BD651, U1 MPU-6000QFN-24, U2 txb0108, Y1 CSTCE16M0V53-R0 16MHZ

Commit message: Minor bugfixes to boards.
Parts:
- Y1: value CSTCE16M0V53-R0 16MHZ -> CSTCE8M00G15C99-R0
Changed lines of the file:
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@@
 <part name="JP18" library="pinhead" deviceset="PINHD-1X9" device=""/>
 <part name="GND21" library="supply1" deviceset="GND" device=""/>
-<part name="Y1" library="SmartPrj" deviceset="RESONATOR" device="MU" value="CSTCE16M0V53-R0 16MHZ"/>
+<part name="Y1" library="SmartPrj" deviceset="RESONATOR" device="MU" value="CSTCE8M00G15C99-R0"/>
 <part name="GND23" library="supply1" deviceset="GND" device=""/>
 <part name="C1" library="SmartPrj" deviceset="C-EU" device="0603-RND" value="100n"/>
@@
 <segment>
 <wire x1="180.34" y1="162.56" x2="165.1" y2="162.56" width="0.1524" layer="91"/>
-<label x="165.1" y="162.56" size="1.778" layer="95"/>
+<label x="167.64" y="162.56" size="1.778" layer="95"/>
 <pinref part="MCU" gate="G$1" pin="P07/D7/AN17"/>
 </segment>
@@
 <segment>
 <wire x1="180.34" y1="165.1" x2="165.1" y2="165.1" width="0.1524" layer="91"/>
-<label x="165.1" y="165.1" size="1.778" layer="95"/>
+<label x="167.64" y="165.1" size="1.778" layer="95"/>
 <pinref part="MCU" gate="G$1" pin="P06/D6/AN16"/>
 </segment>
@@
 <segment>
 <wire x1="180.34" y1="167.64" x2="165.1" y2="167.64" width="0.1524" layer="91"/>
-<label x="165.1" y="167.64" size="1.778" layer="95"/>
+<label x="167.64" y="167.64" size="1.778" layer="95"/>
 <pinref part="MCU" gate="G$1" pin="P05/D5/AN15"/>
 </segment>
@@
 <segment>
 <wire x1="180.34" y1="170.18" x2="165.1" y2="170.18" width="0.1524" layer="91"/>
-<label x="165.1" y="170.18" size="1.778" layer="95"/>
+<label x="167.64" y="170.18" size="1.778" layer="95"/>
 <pinref part="MCU" gate="G$1" pin="P04/D4/AN14"/>
 </segment>

Commit message: Clarifications in schematic
Connections:
- net CS2_3V renamed CS_MOTOR_3V
- net CS_3V renamed CS_GYRO_3V
- net INT2_3V renamed RESET_MOTOR_3V
- net INT_3V renamed INT_GYRO_3V
Changed lines of the file:
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@@
 </segment>
 </net>
-<net name="CS2_3V" class="0">
+<net name="CS_MOTOR_3V" class="0">
 <segment>
 <pinref part="MCU" gate="G$1" pin="P84/INT2"/>
-<wire x1="101.6" y1="127" x2="83.82" y2="127" width="0.1524" layer="91"/>
-<label x="86.36" y="127" size="1.778" layer="95"/>
+<wire x1="101.6" y1="127" x2="81.28" y2="127" width="0.1524" layer="91"/>
+<label x="81.28" y="127" size="1.778" layer="95"/>
 </segment>
 </net>
@@
 <segment>
 <pinref part="MCU" gate="G$1" pin="P81/TA4IN/U/CTS5"/>
-<wire x1="101.6" y1="134.62" x2="83.82" y2="134.62" width="0.1524" layer="91"/>
+<wire x1="101.6" y1="134.62" x2="81.28" y2="134.62" width="0.1524" layer="91"/>
 <label x="86.36" y="134.62" size="1.778" layer="95"/>
 </segment>
@@
 </segment>
 </net>
-<net name="INT2_3V" class="0">
+<net name="RESET_MOTOR_3V" class="0">
 <segment>
 <pinref part="MCU" gate="G$1" pin="P82/INT0"/>
-<wire x1="101.6" y1="132.08" x2="83.82" y2="132.08" width="0.1524" layer="91"/>
-<label x="86.36" y="132.08" size="1.778" layer="95"/>
-</segment>
-</net>
-<net name="CS_3V" class="0">
+<wire x1="101.6" y1="132.08" x2="76.2" y2="132.08" width="0.1524" layer="91"/>
+<label x="76.2" y="132.08" size="1.778" layer="95"/>
+</segment>
+</net>
+<net name="CS_GYRO_3V" class="0">
 <segment>
 <pinref part="MCU" gate="G$1" pin="P83/INT1"/>
-<wire x1="101.6" y1="129.54" x2="83.82" y2="129.54" width="0.1524" layer="91"/>
-<label x="86.36" y="129.54" size="1.778" layer="95"/>
+<wire x1="101.6" y1="129.54" x2="81.28" y2="129.54" width="0.1524" layer="91"/>
+<label x="81.28" y="129.54" size="1.778" layer="95"/>
 </segment>
 </net>
@@
 </segment>
 </net>
-<net name="INT_3V" class="0">
+<net name="INT_GYRO_3V" class="0">
 <segment>
 <pinref part="U1" gate="G$1" pin="INT"/>
-<wire x1="3.81" y1="68.58" x2="-8.89" y2="68.58" width="0.1524" layer="91"/>
-<label x="-8.89" y="68.58" size="1.778" layer="95"/>
+<wire x1="3.81" y1="68.58" x2="-13.97" y2="68.58" width="0.1524" layer="91"/>
+<label x="-13.97" y="68.58" size="1.778" layer="95"/>
 </segment>
 <segment>
@@
 </segment>
 </net>
-<net name="CS_3V" class="0">
+<net name="CS_GYRO_3V" class="0">
 <segment>
 <pinref part="U1" gate="G$1" pin="CS"/>
-<wire x1="39.37" y1="71.12" x2="52.07" y2="71.12" width="0.1524" layer="91"/>
+<wire x1="39.37" y1="71.12" x2="59.69" y2="71.12" width="0.1524" layer="91"/>
 <label x="41.91" y="71.12" size="1.778" layer="95"/>
 </segment>
@@
 <wire x1="128.27" y1="73.66" x2="118.11" y2="73.66" width="0.1524" layer="91"/>
 <pinref part="U2" gate="G$1" pin="A1"/>
-<label x="105.41" y="73.66" size="1.778" layer="95"/>
+<label x="100.33" y="73.66" size="1.778" layer="95"/>
 <pinref part="TP1" gate="G$1" pin="TP"/>
 </segment>
@@
 </segment>
 </net>
-<net name="CS2_3V" class="0">
+<net name="CS_MOTOR_3V" class="0">
 <segment>
 <pinref part="U2" gate="G$1" pin="A7"/>
@@
 </segment>
 </net>
-<net name="INT2_3V" class="0">
+<net name="RESET_MOTOR_3V" class="0">
 <segment>
 <pinref part="U2" gate="G$1" pin="A8"/>
