File: SPI-Gyro-shield/Hardware/Arduino_kuukulgur-alternatiivne2.brd (EAGLE design)
At the start: 99.1 x 53.3 mm, 171 parts, among them IC2 TPS77301DGK, IC4 CP2103_USB_UART, T1 BD651, U1 MPU-6000QFN-24, U2 txb0108, X2 USBSMD, Y1 CSTCE8M00G15C99-R0

Commit message: Misc fixes of nominals
Parts:
- C100, C31: value 47uF/10V -> 100uF/10V
- C29, C30: value 47uF/16V -> 100uF/16V
- C5: value 100n -> 220n
- C7: value 47uF/16V -> 1uF/16V
- LED1: value Red -> Blue
- LED2, LED3, LED4, LED5, LED6: value Green -> Blue
- LED8: value Green -> Red
- R27, R28, R38, R39, R40, R41, R43: value 330r -> 1k
- R35: value (none) -> 100k
- R42: value 1k -> 3k3
- R45: value (none) -> 21k5
- R48: value (none) -> 118k
- R49: value (none) -> 42.2k
