File: SPI-Gyro-shield/Hardware/Arduino_kuukulgur-alternatiivne2.sch (EAGLE design)
At the start: 171 parts, among them IC2 TPS77301DGK, IC4 CP2103_USB_UART, T1 BD651, U1 MPU-6000QFN-24, U2 txb0108, X2 USBSMD, Y1 CSTCE8M00G15C99-R0

Commit message: Misc fixes of nominals
Parts:
- C100, C31: value 47uF/10V -> 100uF/10V
- C29, C30: value 47uF/16V -> 100uF/16V
- C5: value 100n -> 220n
- C7: value 47uF/16V -> 1uF/16V
- LED1: value Red -> Blue
- LED2, LED3, LED4, LED5, LED6: value Green -> Blue
- LED8: value Green -> Red
- R27, R28, R38, R39, R40, R41, R43: value 330r -> 1k
- R35: value (none) -> 100k
- R42: value 1k -> 3k3
- R45: value (none) -> 21k5
- R48: value (none) -> 118k
- R49: value (none) -> 42.2k
Other:
- note added: "Enable at about 7V"
Changed lines of the file:
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@@
 <setting verticaltext="up"/>
 </settings>
-<grid distance="0.05" unitdist="inch" unit="inch" style="lines" multiple="1" display="no" altdistance="0.01" altunitdist="inch" altunit="inch"/>
+<grid distance="0.1" unitdist="inch" unit="inch" style="lines" multiple="1" display="no" altdistance="0.01" altunitdist="inch" altunit="inch"/>
 <layers>
 <layer number="1" name="Top" color="4" fill="1" visible="no" active="no"/>
@@
 <part name="JP12" library="SparkFun" deviceset="M02" device="LOCK"/>
 <part name="S1" library="SparkFun" deviceset="TAC_SWITCH" device="PTH"/>
-<part name="LED1" library="led" deviceset="LED" device="CHIP-LED0603" value="Red"/>
-<part name="LED2" library="led" deviceset="LED" device="CHIP-LED0603" value="Green"/>
+<part name="LED1" library="led" deviceset="LED" device="CHIP-LED0603" value="Blue"/>
+<part name="LED2" library="led" deviceset="LED" device="CHIP-LED0603" value="Blue"/>
 <part name="GND15" library="SparkFun" deviceset="GND" device=""/>
 <part name="GND16" library="SparkFun" deviceset="GND" device=""/>
@@
 <part name="C1" library="SmartPrj" deviceset="C-EU" device="0603-RND" value="100n"/>
 <part name="GND24" library="supply1" deviceset="GND" device=""/>
-<part name="C5" library="SmartPrj" deviceset="C-EU" device="0603-RND" value="100n"/>
+<part name="C5" library="SmartPrj" deviceset="C-EU" device="0603-RND" value="220n"/>
 <part name="C4" library="SmartPrj" deviceset="C-EU" device="0603-RND" value="100n"/>
 <part name="GND25" library="supply1" deviceset="GND" device=""/>
@@
 <part name="JMP1" library="jump-0r-smd" deviceset="0R-JUMP" device="B"/>
 <part name="GND22" library="SparkFun" deviceset="GND" device=""/>
-<part name="R27" library="SmartPrj" deviceset="R-EU_" device="R0603" value="330r"/>
-<part name="R28" library="SmartPrj" deviceset="R-EU_" device="R0603" value="330r"/>
+<part name="R27" library="SmartPrj" deviceset="R-EU_" device="R0603" value="1k"/>
+<part name="R28" library="SmartPrj" deviceset="R-EU_" device="R0603" value="1k"/>
 <part name="U$3" library="tonu" deviceset="TPS54332" device="" value="TPS54332"/>
 <part name="C15" library="SparkFun" deviceset="CAP" device="0603-CAP" value="0.1"/>
@@
 <part name="C9" library="SparkFun" deviceset="CAP" device="0603-CAP" value="180pF"/>
 <part name="C27" library="SparkFun" deviceset="CAP" device="0603-CAP" value="15nF"/>
-<part name="R35" library="SparkFun" deviceset="RESISTOR" device="0603-RES"/>
+<part name="R35" library="SparkFun" deviceset="RESISTOR" device="0603-RES" value="100k"/>
 <part name="R29" library="SparkFun" deviceset="RESISTOR" device="0603-RES" value="63k4"/>
 <part name="R36" library="SparkFun" deviceset="RESISTOR" device="0603-RES" value="1k87"/>
@@
 <part name="D100" library="diode" deviceset="BAT54" device=""/>
 <part name="GND60" library="SparkFun" deviceset="GND" device=""/>
-<part name="C100" library="rcl" deviceset="CPOL-EU" device="C/6032-28R" value="47uF/10V"/>
+<part name="C100" library="rcl" deviceset="CPOL-EU" device="C/6032-28R" value="100uF/10V"/>
 <part name="GND44" library="SparkFun" deviceset="GND" device=""/>
 <part name="L1" library="SparkFun" deviceset="INDUCTOR" device="SRU1038"/>
-<part name="LED3" library="led" deviceset="LED" device="CHIP-LED0603" value="Green"/>
-<part name="R38" library="SmartPrj" deviceset="R-EU_" device="R0603" value="330r"/>
-<part name="R39" library="SmartPrj" deviceset="R-EU_" device="R0603" value="330r"/>
-<part name="R40" library="SmartPrj" deviceset="R-EU_" device="R0603" value="330r"/>
-<part name="R41" library="SmartPrj" deviceset="R-EU_" device="R0603" value="330r"/>
-<part name="LED4" library="led" deviceset="LED" device="CHIP-LED0603" value="Green"/>
-<part name="LED5" library="led" deviceset="LED" device="CHIP-LED0603" value="Green"/>
-<part name="LED6" library="led" deviceset="LED" device="CHIP-LED0603" value="Green"/>
+<part name="LED3" library="led" deviceset="LED" device="CHIP-LED0603" value="Blue"/>
+<part name="R38" library="SmartPrj" deviceset="R-EU_" device="R0603" value="1k"/>
+<part name="R39" library="SmartPrj" deviceset="R-EU_" device="R0603" value="1k"/>
+<part name="R40" library="SmartPrj" deviceset="R-EU_" device="R0603" value="1k"/>
+<part name="R41" library="SmartPrj" deviceset="R-EU_" device="R0603" value="1k"/>
+<part name="LED4" library="led" deviceset="LED" device="CHIP-LED0603" value="Blue"/>
+<part name="LED5" library="led" deviceset="LED" device="CHIP-LED0603" value="Blue"/>
+<part name="LED6" library="led" deviceset="LED" device="CHIP-LED0603" value="Blue"/>
 <part name="GND35" library="supply1" deviceset="GND" device=""/>
 <part name="GND36" library="supply1" deviceset="GND" device=""/>
@@
 </part>
 <part name="LED7" library="led" deviceset="LED" device="CHIP-LED0603" value="Yellow"/>
-<part name="R42" library="SmartPrj" deviceset="R-EU_" device="R0603" value="1k"/>
-<part name="C7" library="rcl" deviceset="C-EU" device="C0805" value="47uF/16V"/>
+<part name="R42" library="SmartPrj" deviceset="R-EU_" device="R0603" value="3k3"/>
+<part name="C7" library="rcl" deviceset="C-EU" device="C0805" value="1uF/16V"/>
 <part name="TP33" library="testpad" deviceset="TP" device="B1,27"/>
 <part name="TP34" library="testpad" deviceset="TP" device="B1,27"/>
@@
 <part name="GND45" library="supply1" deviceset="GND" device=""/>
 <part name="GND46" library="supply1" deviceset="GND" device=""/>
-<part name="R43" library="SmartPrj" deviceset="R-EU_" device="R0603" value="330r"/>
-<part name="LED8" library="led" deviceset="LED" device="CHIP-LED0603" value="Green"/>
+<part name="R43" library="SmartPrj" deviceset="R-EU_" device="R0603" value="1k"/>
+<part name="LED8" library="led" deviceset="LED" device="CHIP-LED0603" value="Red"/>
 <part name="GND47" library="supply1" deviceset="GND" device=""/>
 <part name="IC2" library="samuel" deviceset="TPS773*" device="" value="TPS77301DGK"/>
@@
 <part name="+3V15" library="supply1" deviceset="+3V3" device="" value="+3V3"/>
 <part name="+3V16" library="supply1" deviceset="+3V3" device="" value="+3V3"/>
-<part name="C29" library="rcl" deviceset="CPOL-EU" device="C/6032-28R" value="47uF/16V"/>
+<part name="C29" library="rcl" deviceset="CPOL-EU" device="C/6032-28R" value="100uF/16V"/>
 <part name="+3V17" library="supply1" deviceset="+3V3" device="" value="+3V3"/>
 <part name="GND50" library="supply1" deviceset="GND" device=""/>
-<part name="C30" library="rcl" deviceset="CPOL-EU" device="C/6032-28R" value="47uF/16V"/>
+<part name="C30" library="rcl" deviceset="CPOL-EU" device="C/6032-28R" value="100uF/16V"/>
 <part name="GND51" library="SparkFun" deviceset="GND" device=""/>
-<part name="C31" library="rcl" deviceset="CPOL-EU" device="C/6032-28R" value="47uF/10V"/>
+<part name="C31" library="rcl" deviceset="CPOL-EU" device="C/6032-28R" value="100uF/10V"/>
 <part name="GND52" library="SparkFun" deviceset="GND" device=""/>
 <part name="R44" library="SmartPrj" deviceset="R-EU_" device="R0603" value="47k"/>
 <part name="GND53" library="supply1" deviceset="GND" device=""/>
-<part name="R45" library="SparkFun" deviceset="RESISTOR" device="0603-RES"/>
+<part name="R45" library="SparkFun" deviceset="RESISTOR" device="0603-RES" value="21k5"/>
 <part name="GND54" library="SparkFun" deviceset="GND" device=""/>
 <part name="L4" library="inductor-neosid" deviceset="SM-1206" device="" value="LB3218T220K"/>
@@
 <part name="GND61" library="SparkFun" deviceset="GND" device=""/>
 <part name="GND62" library="SparkFun" deviceset="GND" device=""/>
-<part name="R48" library="rcl" deviceset="R-EU_" device="R0603"/>
-<part name="R49" library="rcl" deviceset="R-EU_" device="R0603"/>
+<part name="R48" library="rcl" deviceset="R-EU_" device="R0603" value="118k"/>
+<part name="R49" library="rcl" deviceset="R-EU_" device="R0603" value="42.2k"/>
 <part name="GND63" library="supply1" deviceset="GND" device=""/>
 </parts>
@@
 <text x="50.8" y="17.78" size="1.778" layer="91">Farnell 1710821</text>
 <text x="50.8" y="15.24" size="1.778" layer="91">Digikey 296-23902-1-ND</text>
+<text x="0" y="20.32" size="1.778" layer="91">Enable at about 7V</text>
 </plain>
 <instances>

Commit message: Cosmetics
Other:
- note added: "http://www.wolframalpha.com/input/?i=%284.5V%2F1.1834V-1%29*42.2kohm"
Changed lines of the file:
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@@
 <attribute name="VALUE" x="64.77" y="169.291" size="1.778" layer="96" rot="R90"/>
 </instance>
-<instance part="+3V11" gate="G$1" x="66.04" y="177.8"/>
-<instance part="+3V13" gate="G$1" x="73.66" y="177.8"/>
+<instance part="+3V11" gate="G$1" x="66.04" y="182.88"/>
+<instance part="+3V13" gate="G$1" x="73.66" y="182.88"/>
 <instance part="R34" gate="G$1" x="-12.7" y="60.96" smashed="yes" rot="R180">
 <attribute name="NAME" x="-16.51" y="62.3316" size="1.778" layer="95"/>
@@
 <wire x1="96.52" y1="53.34" x2="96.52" y2="55.88" width="0.1524" layer="91"/>
 <junction x="96.52" y="55.88"/>
+<label x="88.9" y="55.88" size="1.778" layer="95"/>
 </segment>
 <segment>
@@
 <pinref part="R33" gate="G$1" pin="1"/>
 <pinref part="+3V11" gate="G$1" pin="+3V3"/>
-<wire x1="66.04" y1="175.26" x2="66.04" y2="172.72" width="0.1524" layer="91"/>
+<wire x1="66.04" y1="180.34" x2="66.04" y2="172.72" width="0.1524" layer="91"/>
+<label x="63.5" y="175.26" size="1.778" layer="95" rot="R180"/>
 </segment>
 <segment>
 <pinref part="R32" gate="G$1" pin="1"/>
 <pinref part="+3V13" gate="G$1" pin="+3V3"/>
-<wire x1="73.66" y1="175.26" x2="73.66" y2="172.72" width="0.1524" layer="91"/>
+<wire x1="73.66" y1="180.34" x2="73.66" y2="172.72" width="0.1524" layer="91"/>
+<label x="71.12" y="175.26" size="1.778" layer="95" rot="R180"/>
 </segment>
 </net>
@@
 <pinref part="+3V5" gate="G$1" pin="+3V3"/>
 <wire x1="-20.32" y1="71.12" x2="3.81" y2="71.12" width="0.1524" layer="91"/>
+<label x="-12.7" y="71.12" size="1.778" layer="95"/>
 </segment>
 <segment>
@@
 <sheet>
 <plain>
+<text x="-7.62" y="83.82" size="1.778" layer="91">http://www.wolframalpha.com/input/?i=%284.5V%2F1.1834V-1%29*42.2kohm</text>
 </plain>
 <instances>
