File: SPI-Gyro-shield/Hardware/Arduino_kuukulgur-alternatiivne3.brd (EAGLE design)
At the start: 99.1 x 53.3 mm, 171 parts, among them IC2 TPS77301DGK, IC4 CP2103_USB_UART, T1 BD651, U1 MPU-6000QFN-24, U2 txb0108, X2 USBSMD, Y1 CSTCE8M00G15C99-R0

Commit message: Shield PCB as ordered in.
Parts:
- removed TP34: TPB1,27, testpad:B1,27
- added C34, C35: 1uF/6V, resistor:C0603
- added C36: 100uF/6V, rcl:C/6032-28R
- added C37, C45: 0.1, SparkFun:0603-CAP
- added C38: 10nF, rcl:C0603
- added IC1: TPS77333DGK, samuel:MSOP8
- added IC8: LM2936MP-3.3, national-semiconductor:SOT223
- added TP3: TPB1,27, testpad:B1,27
- added U$1: ASE, crystal:ASE
- C29: value 100uF/16V -> 100uF/6V
- moved TP33 31.5 mm to (77.0, 17.0)
- moved X2 4.00 mm to (4.90, 17.6)
- moved TP43 2.83 mm to (34.8, 13.9)
- moved TP44 2.45 mm to (32.8, 15.3)
- moved C29 2.24 mm to (31.5, 10.0)
- moved C16 1.81 mm to (75.3, 19.5), turned to 270 degrees
- moved S1 1.18 mm to (26.0, 6.12)
- moved L4 1.00 mm to (67.0, 20.2)
- moved C2 0.81 mm to (68.6, 14.0), turned to 90 degrees
Connections:
- removed net _CLK2: MCU.26, R23.1, TP22.TP
- removed net _MISO2: MCU.27, MOTOR2.7, R21.1, R22.2, R33.2, TP24.TP
- removed net _MOSI2: MCU.28, R20.1, R32.2, TP23.TP
- new net +3V3: C12.1, C16.2, C17.2, C33.1, C34.1, C36.+, C37.1, C38.1, IC1.1, IC1.7, IC1.8, IC4.5, IC4.6, IC8.3, JMP1.1, JP3.8, TP33.TP, U$1.1, U$1.4, U1.13, U2.2
- new net CLKIN: U1.1
- new net N$108: MCU.28, R32.2
- new net N$135: MCU.27, R33.2
- new net N$165: MCU.26, TP3.TP
- new net N$166: U$1.3, U1.11
- new net _CLK6: MCU.47, R23.1, TP22.TP
- new net _MISO6: MOTOR2.7, R21.1, R22.2, TP24.TP
- new net _MISO６: MCU.46
- new net _MOSI6: MCU.45, R20.1, TP23.TP
- net +4V5: no longer C12.1, C16.2, C17.2, C33.1, IC4.5, IC4.6, JMP1.1, U1.13, U2.2
- net +5V: now also C35.1, C45.1, IC1.5, IC1.6, IC8.1
- net GND: now also C34.2, C35.2, C36.-, C37.2, C38.2, C45.2, IC1.3, IC1.4, IC8.2, IC8.4, U$1.2; no longer U1.1
- net RX3: no longer MCU.45, TP33.TP
- net TX3: no longer MCU.46, TP34.TP
Routing:
- net GND: track 563.7 -> 299.2 mm, vias 176 -> 117
- net +4V5: track 260.2 -> 104.8 mm, vias 10 -> 7
- net +3V3: track 0.00 -> 137.4 mm, vias 0 -> 5
- net _MISO6: track 0.00 -> 47.5 mm, vias 0 -> 2
- net RX3: track 42.8 -> 0.00 mm, vias 1 -> 0
- net TX3: track 39.9 -> 0.00 mm, vias 1 -> 0
- net _MOSI6: track 0.00 -> 29.0 mm, vias 0 -> 2
- net _CLK6: track 0.00 -> 26.3 mm, vias 0 -> 2
- net _MOSI2: track 25.8 -> 0.00 mm
- net _MISO2: track 25.8 -> 0.00 mm, vias 1 -> 0
- net +5V: track 178.2 -> 197.5 mm, vias 2 -> 3
- net _CLK2: track 17.2 -> 0.00 mm
- net +5V_A: track 48.6 -> 34.2 mm, vias 1 -> 0
- net RESET: track 95.5 -> 82.0 mm
- net WR: track 58.8 -> 45.6 mm
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
Commit message: Misc schematic clarifications
Connections:
- net CLK1 renamed CLK4
- net CS1 renamed CS4
- net MOSI1 renamed MOSI4
Changed lines of the file:
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@@
 <layer number="14" name="Route14" color="1" fill="6" visible="no" active="yes"/>
 <layer number="15" name="Route15" color="4" fill="6" visible="no" active="yes"/>
-<layer number="16" name="Bottom" color="1" fill="1" visible="no" active="yes"/>
+<layer number="16" name="Bottom" color="1" fill="1" visible="yes" active="yes"/>
 <layer number="17" name="Pads" color="2" fill="1" visible="yes" active="yes"/>
 <layer number="18" name="Vias" color="14" fill="1" visible="yes" active="yes"/>
@@
 <wire x1="24.9176" y1="37.9978" x2="24.5" y2="37.5802" width="0.2032" layer="15"/>
 </signal>
-<signal name="CS1">
+<signal name="CS4">
 <contactref element="MOTOR1" pad="1"/>
 <contactref element="R7" pad="2"/>
@@
 <wire x1="47.0785" y1="28.73" x2="48.12" y2="28.73" width="0.2032" layer="1"/>
 </signal>
-<signal name="CLK1">
+<signal name="CLK4">
 <contactref element="MOTOR1" pad="3"/>
 <contactref element="R6" pad="2"/>
@@
 <wire x1="50.66" y1="27.6885" x2="50.66" y2="28.73" width="0.2032" layer="1"/>
 </signal>
-<signal name="MOSI1">
+<signal name="MOSI4">
 <contactref element="MOTOR1" pad="5"/>
 <contactref element="R1" pad="2"/>
