File: PowerSupply/Hardware/kulgurpower2.brd (EAGLE design)
At the start: 102 x 86.5 mm, 154 parts, among them M1 MST2V, M2 MST2V, M3 MST2V, M4 MST2V, X1 1727036, X2 2534-, X3 22-23-2031, X4 22-23-2031, X5 22-23-2021

Commit message: New lower PCB of power supply in
Parts:
- added Q1, Q2, Q3, Q4: BSH103, adafruit:SOT23
- added R27, R30, R34, R37, R38, R43, R44, R47: 430k, rcl:R0603
- added R28, R29, R35, R36, R41, R42, R45, R46: 100k, rcl:R0603
- moved D4 1.89 mm to (20.5, 48.9)
- moved C28 1.80 mm to (45.2, 16.8)
- moved C27 1.52 mm to (33.6, 16.8)
- moved C26 1.41 mm to (22.2, 16.8)
- moved C25 1.12 mm to (10.0, 16.8)
Connections:
- net !OFF_0: now also Q1.3, R27.1, R28.2
- net !OFF_1: now also Q2.3, R34.1, R35.2
- net !OFF_2: now also Q3.3, R38.1, R41.2
- net !OFF_3: now also Q4.3, R44.1, R45.2
- net BAT0_EN: now also Q1.1, R29.2, R30.1
- net BAT1_EN: now also Q2.1, R36.2, R37.1
- net BAT2_EN: now also Q3.1, R42.2, R43.1
- net BAT3_EN: now also Q4.1, R46.2, R47.1
- net GND: now also Q1.2, Q2.2, Q3.2, Q4.2, R28.1, R29.1, R35.1, R36.1, R41.1, R42.1, R45.1, R46.1
- net VBAT0_X: now also R27.2, R30.2
- net VBAT1_X: now also R34.2, R37.2
- net VBAT2_X: now also R38.2, R43.2
- net VBAT3_X: now also R44.2, R47.2
Routing:
- net GND: track 74.9 -> 288.2 mm, vias 91 -> 49
- net !OFF_2: track 0.65 -> 26.5 mm, vias 0 -> 2
- net !OFF_1: track 2.66 -> 27.1 mm, vias 0 -> 2
- net +5V: track 55.5 -> 33.0 mm, vias 4 -> 2
- net !OFF_3: track 0.65 -> 21.8 mm, vias 0 -> 3
- net !OFF_0: track 2.66 -> 21.4 mm, vias 0 -> 2
- net OUT2_S: track 13.8 -> 0.76 mm
- net BAT3_EN: track 35.3 -> 48.4 mm, vias 2 -> 1
- net VBAT2_X: track 52.1 -> 64.7 mm, vias 2 -> 1
- net BAT2_EN: track 32.5 -> 42.2 mm, vias 2 -> 3
- net VBAT3_X: track 60.0 -> 68.9 mm
- net OUT3_S: track 11.4 -> 2.82 mm
- net X1: track 19.6 -> 11.7 mm
- net IMON1: track 56.9 -> 49.2 mm
- net VBAT1_X: track 58.7 -> 51.9 mm
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- removed copper zone on layer 1, net BAT-
- removed copper zone on layer 1, net GND
- removed copper zone on layer 2, net GND
