File: PowerSupply/Hardware/kulgurpower2.sch (EAGLE design)
At the start: 154 parts, among them M1 MST2V, M2 MST2V, M3 MST2V, M4 MST2V, X1 1727036, X2 2534-, X3 22-23-2031, X4 22-23-2031, X5 22-23-2021

Commit message: New lower PCB of power supply in
Parts:
- added Q1, Q2, Q3, Q4: BSH103, adafruit:MOSFET-NREFLOW
- added R27, R30, R34, R37, R38, R43, R44, R47: 430k, rcl:R-EU_R0603
- added R28, R29, R35, R36, R41, R42, R45, R46: 100k, rcl:R-EU_R0603
Connections:
- net !OFF_0: now also Q1.D, R27.1, R28.2
- net !OFF_1: now also Q2.D, R34.1, R35.2
- net !OFF_2: now also Q3.D, R38.1, R41.2
- net !OFF_3: now also Q4.D, R44.1, R45.2
- net BAT0_EN: now also Q1.G, R29.2, R30.1
- net BAT1_EN: now also Q2.G, R36.2, R37.1
- net BAT2_EN: now also Q3.G, R42.2, R43.1
- net BAT3_EN: now also Q4.G, R46.2, R47.1
- net GND: now also Q1.S, Q2.S, Q3.S, Q4.S, R28.1, R29.1, R35.1, R36.1, R41.1, R42.1, R45.1, R46.1
- net VBAT0_X: now also R27.2, R30.2
- net VBAT1_X: now also R34.2, R37.2
- net VBAT2_X: now also R38.2, R43.2
- net VBAT3_X: now also R44.2, R47.2
Other:
- note added: "Resistor dividers keep voltage in reasonable range"
- note added: "Transistor reverses input signal"
- note removed: "MOSFET drivers"
