File: PowerSupply/Hardware/kulgurpower.brd (EAGLE design)
At the start: 102 x 86.5 mm, 138 parts, among them M1 MST2V, M2 MST2V, M3 MST2V, M4 MST2V, X1 1727036, X2 2534-, X3 22-23-2031, X4 22-23-2031, X5 22-23-2021

Commit message: Minor fixes to PCB
Parts:
- removed C13, C14: (no value), rcl:C/6032-28R
- added C31, C35: (no value), rcl:C/6032-28R
- added C36, C37: 15V, rcl:C/6032-28R
- added C38: 15V, rcl:175TMP-0810
- added C39: 15v, rcl:175TMP-0810
- added D4: MBRS330T3, diode:SMC
- added PAD1, PAD2, PAD3, PAD4, PAD5, PAD6, PAD7, PAD8: (no value), wirepad:1,6/0,9
- C104, C113, C32: value 220n -> 0.1
- C3: value (none) -> 15V
- L1, L2: device inductors:DR73 -> inductors:DR125
- moved C10 7.95 mm to (82.8, 43.3)
- moved U$17 7.02 mm to (83.7, 34.6)
- moved L2 6.81 mm to (72.0, 17.0), turned to 270 degrees
- moved SJ104 6.72 mm to (77.3, 33.0)
- moved C1 6.72 mm to (94.6, 28.6)
- moved C16 6.72 mm to (90.3, 34.3)
- moved C17 6.72 mm to (72.7, 36.0)
- moved C2 6.72 mm to (72.6, 28.6)
- moved C20 6.72 mm to (77.3, 34.3)
- moved C21 6.72 mm to (81.4, 28.2)
- moved C29 6.72 mm to (85.1, 20.3)
- moved C33 6.72 mm to (82.2, 41.5)
- moved C5 6.72 mm to (83.7, 24.4)
- moved R21 6.72 mm to (90.3, 36.4)
- moved R23 6.72 mm to (85.3, 39.3)
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Connections:
- net 5V renamed 5V_LDO
- new net +19V_CHG: D4.C, X2.14, X2.16
- new net N$2: D4.A
- net +19V: no longer X2.14, X2.16
- net +5V: now also C31.+, C35.+; no longer C13.+
- net GND: now also C31.-, C35.-, C36.-, C37.-, C38.-, C39.-; no longer C13.-, C14.-
- net SERVO: no longer C14.+
- net V+: now also C36.+, C37.+, C38.+, C39.+
- net VBAT0: no longer X2.1, X2.2
- net VBAT0_X: now also PAD1.1, PAD8.1, X2.1, X2.2
- net VBAT1: no longer X2.3, X2.4
- net VBAT1_X: now also PAD2.1, PAD7.1, X2.3, X2.4
- net VBAT2: no longer X2.5, X2.6
- net VBAT2_X: now also PAD3.1, PAD6.1, X2.5, X2.6
- net VBAT3: no longer X2.7, X2.8
- net VBAT3_X: now also PAD4.1, PAD5.1, X2.7, X2.8
Routing:
- net VBAT3: track 61.2 -> 0.00 mm, vias 2 -> 0
- net VBAT2: track 53.1 -> 0.00 mm, vias 3 -> 0
- net VBAT3_X: track 15.8 -> 60.0 mm
- net VBAT1_X: track 16.1 -> 58.7 mm
- net VBAT1: track 40.1 -> 0.00 mm, vias 2 -> 0
- net VBAT0: track 40.0 -> 0.00 mm, vias 1 -> 0
- net VBAT0_X: track 15.1 -> 47.5 mm
- net VBAT2_X: track 20.0 -> 52.1 mm
- net +5V: track 27.6 -> 55.5 mm, vias 2 -> 4
- net SERVO: track 16.9 -> 39.6 mm, vias 4 -> 8
- net GND: track 47.1 -> 64.6 mm, vias 60 -> 92
- net X2: track 3.82 -> 18.3 mm, vias 2 -> 1
- net X1: track 5.22 -> 19.6 mm, vias 2 -> 1
- net OUT2_S: track 0.79 -> 13.8 mm
- net +19V_CHG: track 0.00 -> 13.0 mm, vias 0 -> 1
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- added copper zone on layer 15, net +5V

Commit message: Two resistors in ladder were swapped Nominals rised for pullup. Next power bill will be smaller!
Parts:
- R10, R14: value 100k -> 430k
Changed lines of the file:
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@@
 <layer number="20" name="Dimension" color="15" fill="1" visible="yes" active="yes"/>
 <layer number="21" name="tPlace" color="7" fill="1" visible="no" active="yes"/>
-<layer number="22" name="bPlace" color="7" fill="1" visible="no" active="yes"/>
+<layer number="22" name="bPlace" color="7" fill="1" visible="yes" active="yes"/>
 <layer number="23" name="tOrigins" color="15" fill="1" visible="yes" active="yes"/>
 <layer number="24" name="bOrigins" color="15" fill="1" visible="yes" active="yes"/>
 <layer number="25" name="tNames" color="7" fill="1" visible="no" active="yes"/>
-<layer number="26" name="bNames" color="7" fill="1" visible="no" active="yes"/>
+<layer number="26" name="bNames" color="7" fill="1" visible="yes" active="yes"/>
 <layer number="27" name="tValues" color="7" fill="1" visible="no" active="yes"/>
-<layer number="28" name="bValues" color="7" fill="1" visible="no" active="yes"/>
+<layer number="28" name="bValues" color="7" fill="1" visible="yes" active="yes"/>
 <layer number="29" name="tStop" color="7" fill="3" visible="no" active="yes"/>
-<layer number="30" name="bStop" color="7" fill="6" visible="no" active="yes"/>
+<layer number="30" name="bStop" color="7" fill="6" visible="yes" active="yes"/>
 <layer number="31" name="tCream" color="7" fill="4" visible="no" active="yes"/>
-<layer number="32" name="bCream" color="7" fill="5" visible="no" active="yes"/>
+<layer number="32" name="bCream" color="7" fill="5" visible="yes" active="yes"/>
 <layer number="33" name="tFinish" color="6" fill="3" visible="no" active="yes"/>
-<layer number="34" name="bFinish" color="6" fill="6" visible="no" active="yes"/>
+<layer number="34" name="bFinish" color="6" fill="6" visible="yes" active="yes"/>
 <layer number="35" name="tGlue" color="7" fill="4" visible="no" active="yes"/>
-<layer number="36" name="bGlue" color="7" fill="5" visible="no" active="yes"/>
+<layer number="36" name="bGlue" color="7" fill="5" visible="yes" active="yes"/>
 <layer number="37" name="tTest" color="7" fill="1" visible="no" active="yes"/>
-<layer number="38" name="bTest" color="7" fill="1" visible="no" active="yes"/>
+<layer number="38" name="bTest" color="7" fill="1" visible="yes" active="yes"/>
 <layer number="39" name="tKeepout" color="4" fill="11" visible="no" active="yes"/>
-<layer number="40" name="bKeepout" color="1" fill="11" visible="no" active="yes"/>
+<layer number="40" name="bKeepout" color="1" fill="11" visible="yes" active="yes"/>
 <layer number="41" name="tRestrict" color="4" fill="10" visible="no" active="yes"/>
-<layer number="42" name="bRestrict" color="1" fill="10" visible="no" active="yes"/>
+<layer number="42" name="bRestrict" color="1" fill="10" visible="yes" active="yes"/>
 <layer number="43" name="vRestrict" color="2" fill="10" visible="no" active="yes"/>
 <layer number="44" name="Drills" color="7" fill="1" visible="no" active="yes"/>
@@
 <layer number="50" name="dxf" color="7" fill="1" visible="no" active="no"/>
 <layer number="51" name="tDocu" color="7" fill="1" visible="no" active="yes"/>
-<layer number="52" name="bDocu" color="7" fill="1" visible="no" active="yes"/>
+<layer number="52" name="bDocu" color="7" fill="1" visible="yes" active="yes"/>
 <layer number="53" name="tGND_GNDA" color="7" fill="9" visible="no" active="no"/>
 <layer number="54" name="bGND_GNDA" color="1" fill="9" visible="no" active="no"/>
@@
 <attribute name="OC_FARNELL" value="1462926" x="75" y="82" size="1.778" layer="27" rot="R270" display="off"/>
 </element>
-<element name="R10" library="rcl" package="R0603" value="100k" x="67.898" y="36.7124" smashed="yes" rot="R90"/>
-<element name="R14" library="rcl" package="R0603" value="100k" x="65.6882" y="36.7124" smashed="yes" rot="R90"/>
+<element name="R10" library="rcl" package="R0603" value="430k" x="67.898" y="36.7124" smashed="yes" rot="R90"/>
+<element name="R14" library="rcl" package="R0603" value="430k" x="65.6882" y="36.7124" smashed="yes" rot="R90"/>
 <element name="C15" library="rcl" package="C/6032-28R" value="" x="72.0198" y="17.0435" smashed="yes" rot="MR270">
 <attribute name="VALUE" x="75.0698" y="20.0435" size="1.27" layer="28" rot="MR270"/>

Commit message: PCB updates
Parts:
- C11, C18, C4, C7: value 0.1 -> 1n
- R25, R33: value 100k -> 3k9
- R31, R32: value 3k16 -> 10k
- R39: value 30k -> 24k
- R40: value 270k -> 143k
- R5: value 30k -> 24.3
Changed lines of the file:
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@@
 <layers>
 <layer number="1" name="Top" color="4" fill="1" visible="yes" active="yes"/>
-<layer number="2" name="Route2" color="1" fill="3" visible="no" active="yes"/>
+<layer number="2" name="Route2" color="1" fill="3" visible="yes" active="yes"/>
 <layer number="3" name="Route3" color="4" fill="3" visible="no" active="no"/>
 <layer number="4" name="Route4" color="1" fill="4" visible="no" active="no"/>
@@
 <layer number="13" name="Route13" color="4" fill="5" visible="no" active="no"/>
 <layer number="14" name="Route14" color="1" fill="6" visible="no" active="no"/>
-<layer number="15" name="Route15" color="4" fill="6" visible="no" active="yes"/>
+<layer number="15" name="Route15" color="4" fill="6" visible="yes" active="yes"/>
 <layer number="16" name="Bottom" color="1" fill="1" visible="yes" active="yes"/>
 <layer number="17" name="Pads" color="2" fill="1" visible="yes" active="yes"/>
@@
 <layer number="19" name="Unrouted" color="6" fill="1" visible="yes" active="yes"/>
 <layer number="20" name="Dimension" color="15" fill="1" visible="yes" active="yes"/>
-<layer number="21" name="tPlace" color="7" fill="1" visible="no" active="yes"/>
+<layer number="21" name="tPlace" color="7" fill="1" visible="yes" active="yes"/>
 <layer number="22" name="bPlace" color="7" fill="1" visible="yes" active="yes"/>
 <layer number="23" name="tOrigins" color="15" fill="1" visible="yes" active="yes"/>
 <layer number="24" name="bOrigins" color="15" fill="1" visible="yes" active="yes"/>
-<layer number="25" name="tNames" color="7" fill="1" visible="no" active="yes"/>
+<layer number="25" name="tNames" color="7" fill="1" visible="yes" active="yes"/>
 <layer number="26" name="bNames" color="7" fill="1" visible="yes" active="yes"/>
-<layer number="27" name="tValues" color="7" fill="1" visible="no" active="yes"/>
+<layer number="27" name="tValues" color="7" fill="1" visible="yes" active="yes"/>
 <layer number="28" name="bValues" color="7" fill="1" visible="yes" active="yes"/>
-<layer number="29" name="tStop" color="7" fill="3" visible="no" active="yes"/>
+<layer number="29" name="tStop" color="7" fill="3" visible="yes" active="yes"/>
 <layer number="30" name="bStop" color="7" fill="6" visible="yes" active="yes"/>
-<layer number="31" name="tCream" color="7" fill="4" visible="no" active="yes"/>
+<layer number="31" name="tCream" color="7" fill="4" visible="yes" active="yes"/>
 <layer number="32" name="bCream" color="7" fill="5" visible="yes" active="yes"/>
-<layer number="33" name="tFinish" color="6" fill="3" visible="no" active="yes"/>
+<layer number="33" name="tFinish" color="6" fill="3" visible="yes" active="yes"/>
 <layer number="34" name="bFinish" color="6" fill="6" visible="yes" active="yes"/>
-<layer number="35" name="tGlue" color="7" fill="4" visible="no" active="yes"/>
+<layer number="35" name="tGlue" color="7" fill="4" visible="yes" active="yes"/>
 <layer number="36" name="bGlue" color="7" fill="5" visible="yes" active="yes"/>
-<layer number="37" name="tTest" color="7" fill="1" visible="no" active="yes"/>
+<layer number="37" name="tTest" color="7" fill="1" visible="yes" active="yes"/>
 <layer number="38" name="bTest" color="7" fill="1" visible="yes" active="yes"/>
-<layer number="39" name="tKeepout" color="4" fill="11" visible="no" active="yes"/>
+<layer number="39" name="tKeepout" color="4" fill="11" visible="yes" active="yes"/>
 <layer number="40" name="bKeepout" color="1" fill="11" visible="yes" active="yes"/>
-<layer number="41" name="tRestrict" color="4" fill="10" visible="no" active="yes"/>
+<layer number="41" name="tRestrict" color="4" fill="10" visible="yes" active="yes"/>
 <layer number="42" name="bRestrict" color="1" fill="10" visible="yes" active="yes"/>
 <layer number="43" name="vRestrict" color="2" fill="10" visible="no" active="yes"/>
@@
 <element name="U$3" library="FDMS8558S" package="POWER56" value="AON6500" x="50.0212" y="19.1503" rot="MR180"/>
 <element name="U$4" library="SparkFun-AnalogIC" package="SO08" value="ACS712" x="47.5787" y="12.632" smashed="yes" rot="MR270"/>
-<element name="C7" library="rcl" package="C0603" value="0.1" x="42.4033" y="11.1381" smashed="yes" rot="MR90"/>
+<element name="C7" library="rcl" package="C0603" value="1n" x="42.4033" y="11.1381" smashed="yes" rot="MR90"/>
 <element name="U$6" library="FDMS8558S" package="POWER56" value="AON6500" x="38.554" y="26.046" rot="MR0"/>
 <element name="U$7" library="FDMS8558S" package="POWER56" value="AON6500" x="38.554" y="19.158" rot="MR180"/>
 <element name="U$8" library="SparkFun-AnalogIC" package="SO08" value="ACS712" x="35.9029" y="12.597" smashed="yes" rot="MR270"/>
-<element name="C4" library="rcl" package="C0603" value="0.1" x="30.8968" y="11.1075" smashed="yes" rot="MR90"/>
+<element name="C4" library="rcl" package="C0603" value="1n" x="30.8968" y="11.1075" smashed="yes" rot="MR90"/>
 <element name="U$9" library="FDMS8558S" package="POWER56" value="AON6500" x="26.995" y="26.046" rot="MR0"/>
 <element name="U$10" library="FDMS8558S" package="POWER56" value="AON6500" x="26.995" y="19.158" rot="MR180"/>
 <element name="U$11" library="SparkFun-AnalogIC" package="SO08" value="ACS712" x="24.3778" y="12.6495" smashed="yes" rot="MR270"/>
-<element name="C11" library="rcl" package="C0603" value="0.1" x="19.4325" y="11.1545" smashed="yes" rot="MR90"/>
+<element name="C11" library="rcl" package="C0603" value="1n" x="19.4325" y="11.1545" smashed="yes" rot="MR90"/>
 <element name="U$5" library="FDMS8558S" package="POWER56" value="AON6500" x="15.047" y="26.046" rot="MR0"/>
 <element name="U$12" library="FDMS8558S" package="POWER56" value="AON6500" x="15.047" y="19.158" rot="MR180"/>
 <element name="U$13" library="SparkFun-AnalogIC" package="SO08" value="ACS712" x="12.3581" y="12.6458" smashed="yes" rot="MR270"/>
-<element name="C18" library="rcl" package="C0603" value="0.1" x="7.224" y="11.1126" smashed="yes" rot="MR90"/>
+<element name="C18" library="rcl" package="C0603" value="1n" x="7.224" y="11.1126" smashed="yes" rot="MR90"/>
 <element name="PC" library="con-phoenix-508" package="MSTBV2" value="MST2V" x="84.25" y="81.75" smashed="yes">
 <attribute name="NAME" x="82.535" y="75.654" size="1.778" layer="25" ratio="10"/>
@@
 <element name="U$17" library="tps51222" package="QFN-32" value="TPS51222RTVT" x="83.7215" y="34.5885" rot="R90"/>
 <element name="R3" library="rcl" package="R0603" value="300k" x="86.5446" y="25.6307" smashed="yes" rot="R90"/>
-<element name="R39" library="rcl" package="R0603" value="30k" x="82.1765" y="39.3427" smashed="yes" rot="R180"/>
+<element name="R39" library="rcl" package="R0603" value="24k" x="82.1765" y="39.3427" smashed="yes" rot="R180"/>
 <element name="R23" library="rcl" package="R0603" value="18k" x="85.2725" y="39.3453" smashed="yes" rot="R180"/>
 <element name="R4" library="rcl" package="R0603" value="30k" x="90.268" y="38.4427" smashed="yes" rot="R180"/>
-<element name="R5" library="rcl" package="R0603" value="30k" x="77.2929" y="38.4604" smashed="yes"/>
+<element name="R5" library="rcl" package="R0603" value="24.3" x="77.2929" y="38.4604" smashed="yes"/>
 <element name="R21" library="rcl" package="R0603" value="120k" x="90.2688" y="36.3686" smashed="yes"/>
-<element name="R40" library="rcl" package="R0603" value="270k" x="77.2749" y="36.3829" smashed="yes" rot="R180"/>
+<element name="R40" library="rcl" package="R0603" value="143k" x="77.2749" y="36.3829" smashed="yes" rot="R180"/>
 <element name="C5" library="rcl" package="C1210" value="10u" x="83.6737" y="24.4193" smashed="yes" rot="R90"/>
 <element name="C21" library="rcl" package="C0603" value="0,1u" x="81.396" y="28.2134" smashed="yes" rot="R180"/>
@@
 <element name="C17" library="rcl" package="C1210" value="10uF/6.3V" x="72.7084" y="35.9885" smashed="yes" rot="R270"/>
 <element name="SJ104" library="rcl" package="R0603" value="0R" x="77.2764" y="32.9714" smashed="yes" rot="MR0"/>
-<element name="R31" library="rcl" package="R0603" value="3k16" x="88.6898" y="29.6644" smashed="yes" rot="R270"/>
-<element name="R32" library="rcl" package="R0603" value="3k16" x="78.8404" y="29.643" smashed="yes" rot="R270"/>
-<element name="R25" library="rcl" package="R0603" value="100k" x="90.2637" y="32.2263" smashed="yes"/>
+<element name="R31" library="rcl" package="R0603" value="10k" x="88.6898" y="29.6644" smashed="yes" rot="R270"/>
+<element name="R32" library="rcl" package="R0603" value="10k" x="78.8404" y="29.643" smashed="yes" rot="R270"/>
+<element name="R25" library="rcl" package="R0603" value="3k9" x="90.2637" y="32.2263" smashed="yes"/>
 <element name="C16" library="rcl" package="C0603" value="0,1u" x="90.27" y="34.299" smashed="yes" rot="R180"/>
-<element name="R33" library="rcl" package="R0603" value="100k" x="77.2689" y="32.2297" smashed="yes"/>
+<element name="R33" library="rcl" package="R0603" value="3k9" x="77.2689" y="32.2297" smashed="yes"/>
 <element name="C20" library="rcl" package="C0603" value="0,1u" x="77.2747" y="34.3119" smashed="yes"/>
 <element name="SJ114" library="rcl" package="R0603" value="0R" x="90.7584" y="29.6682" smashed="yes" rot="R270"/>
