File: PowerSupply/Hardware/kulgurpowerMCU3-unrouted.brd (EAGLE design)
At the start: 102 x 57 mm, 150 parts, among them U1 MPU-6000QFN-24, U2 MPU-6000QFN-24, X1 12Mhz, X2 2534-, X3 22-23-2021

Commit message: PCB updates
Parts:
- moved AN0 0.50 mm to (55.0, 36.4)
Routing:
- net AN0: track 33.3 -> 32.8 mm
- net GND: vias 185 -> 184
Changed lines of the file:
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@@
 <layer number="20" name="Dimension" color="15" fill="1" visible="yes" active="yes"/>
 <layer number="21" name="tPlace" color="7" fill="1" visible="yes" active="yes"/>
-<layer number="22" name="bPlace" color="7" fill="1" visible="no" active="yes"/>
+<layer number="22" name="bPlace" color="7" fill="1" visible="yes" active="yes"/>
 <layer number="23" name="tOrigins" color="15" fill="1" visible="yes" active="yes"/>
-<layer number="24" name="bOrigins" color="15" fill="1" visible="no" active="yes"/>
+<layer number="24" name="bOrigins" color="15" fill="1" visible="yes" active="yes"/>
 <layer number="25" name="tNames" color="7" fill="1" visible="yes" active="yes"/>
-<layer number="26" name="bNames" color="7" fill="1" visible="no" active="yes"/>
-<layer number="27" name="tValues" color="7" fill="1" visible="no" active="yes"/>
-<layer number="28" name="bValues" color="7" fill="1" visible="no" active="yes"/>
+<layer number="26" name="bNames" color="7" fill="1" visible="yes" active="yes"/>
+<layer number="27" name="tValues" color="7" fill="1" visible="yes" active="yes"/>
+<layer number="28" name="bValues" color="7" fill="1" visible="yes" active="yes"/>
 <layer number="29" name="tStop" color="7" fill="3" visible="no" active="yes"/>
 <layer number="30" name="bStop" color="7" fill="6" visible="no" active="yes"/>
@@
 </element>
 <element name="C12" library="SparkFun" package="0603-CAP" value="0.1" x="56.0257" y="34.3957" smashed="yes" rot="R270"/>
-<element name="AN0" library="testpad" package="B1,27" value="TPB1,27" x="55.0467" y="36.9215" smashed="yes" rot="R90">
-<attribute name="TP_SIGNAL_NAME" value="" x="56.9517" y="36.2865" size="1" layer="37" rot="R90"/>
+<element name="AN0" library="testpad" package="B1,27" value="TPB1,27" x="55.0467" y="36.4215" smashed="yes" rot="R90">
+<attribute name="TP_SIGNAL_NAME" value="" x="56.9517" y="35.7865" size="1" layer="37" rot="R90"/>
 </element>
 <element name="R18" library="rcl" package="R0603" value="100k" x="53.9152" y="34.4035" smashed="yes" rot="R270"/>
@@
 <element name="D1" library="diode" package="SMC" value="MBRS320T3" x="28.544" y="53.0799" smashed="yes" rot="MR0"/>
 <element name="C50" library="rcl" package="C1210" value="22uF/25V" x="36.75" y="54.75" smashed="yes" rot="MR180"/>
-<element name="U$4" library="crystal" package="ASE" value="ASE" x="53.25" y="17">
+<element name="U$4" library="crystal" package="ASE" value="ASE" x="53.25" y="17" smashed="yes">
 <attribute name="OC_NEWARK" value="unknown" x="53.25" y="17" size="1.778" layer="27" display="off"/>
 <attribute name="MPN" value="" x="53.25" y="17" size="1.778" layer="27" display="off"/>
@@
 <attribute name="OC_FARNELL" value="unknown" x="53.25" y="17" size="1.778" layer="27" display="off"/>
 </element>
-<element name="TP1" library="testpad" package="B1,27" value="TPB1,27" x="50.75" y="15.5">
-<attribute name="TP_SIGNAL_NAME" value="" x="50.75" y="15.5" size="1.778" layer="27" display="off"/>
+<element name="TP1" library="testpad" package="B1,27" value="TPB1,27" x="50.75" y="15.5" smashed="yes">
+<attribute name="TP_SIGNAL_NAME" value="" x="50.115" y="13.595" size="1" layer="37"/>
+<attribute name="VALUE" x="50.115" y="14.738" size="0.0254" layer="27"/>
 </element>
-<element name="U$6" library="XCL202" package="CL2025" value="XCL202B331BR-G" x="50.25" y="45.75" rot="R90"/>
-<element name="C53" library="rcl" package="C0603" value="10uF / 6.3V" x="52.75" y="45.75" rot="R90"/>
-<element name="C54" library="rcl" package="C0603" value="4.7uF / 10V" x="47.75" y="45.75" rot="R270"/>
+<element name="U$6" library="XCL202" package="CL2025" value="XCL202B331BR-G" x="50.25" y="45.75" smashed="yes" rot="R90">
+<attribute name="NAME" x="52.25" y="43.75" size="0.8128" layer="51" rot="R180"/>
+<attribute name="VALUE" x="52.25" y="48.25" size="0.8128" layer="51" rot="R180"/>
+</element>
+<element name="C53" library="rcl" package="C0603" value="10uF / 6.3V" x="52.75" y="45.75" smashed="yes" rot="R90"/>
+<element name="C54" library="rcl" package="C0603" value="4.7uF / 10V" x="47.75" y="45.75" smashed="yes" rot="R270"/>
 <element name="U$5" library="tonu" package="SO8" value="TPS54332" x="17.5" y="14.25" smashed="yes" rot="MR90"/>
 <element name="C28" library="SparkFun" package="0603-CAP" value="0.1" x="14.5" y="10.75" smashed="yes" rot="MR0"/>
@@
 <element name="C58" library="rcl" package="C/6032-28R" value="100uF/16V" x="6.9767" y="8.0394" smashed="yes" rot="MR90"/>
 <element name="R45" library="SparkFun" package="0603-RES" value="21k5" x="11.25" y="17.25" smashed="yes" rot="MR180"/>
-<element name="L7" library="inductors" package="DR73" value="4,7uH" x="26.0374" y="6.3985" rot="MR270"/>
+<element name="L7" library="inductors" package="DR73" value="4,7uH" x="26.0374" y="6.3985" smashed="yes" rot="MR270">
+<attribute name="NAME" x="22.0374" y="9.8985" size="1.27" layer="26" rot="MR270"/>
+</element>
 </elements>
 <signals>
@@
 <via x="6.97933125" y="5.4862" extent="1-16" drill="0.6" diameter="0.6096"/>
 <via x="24.138159375" y="11.41869375" extent="1-16" drill="0.3048" diameter="0.6096"/>
-<via x="25.138159375" y="11.41869375" extent="1-16" drill="0.3048" diameter="0.6096"/>
+<wire x1="25.138159375" y1="11.41869375" x2="25.138159375" y2="11.41869375" width="0" layer="19" extent="1-16"/>
 <via x="28.638159375" y="10.66869375" extent="1-16" drill="0.3048" diameter="0.6096"/>
 <via x="28.638159375" y="9.66869375" extent="1-16" drill="0.3048" diameter="0.6096"/>
@@
 <wire x1="55.5952" y1="32.4704" x2="51.6248" y2="28.5" width="0.2032" layer="1"/>
 <wire x1="51.6248" y1="28.5" x2="31.8453" y2="28.5" width="0.2032" layer="1"/>
-<wire x1="31.8453" y1="28.5" x2="31.0358" y2="27.6905" width="0.2032" layer="1"/>
-<wire x1="31.0358" y1="27.6905" x2="31.0358" y2="27.3224" width="0.2032" layer="1"/>
-<wire x1="31.0358" y1="27.3224" x2="29.9175" y2="26.2041" width="0.2032" layer="1"/>
+<wire x1="31.8453" y1="28.5" x2="30.7858" y2="27.4405" width="0.2032" layer="1"/>
+<wire x1="30.7858" y1="27.4405" x2="30.7858" y2="27.0724" width="0.2032" layer="1"/>
+<wire x1="30.7858" y1="27.0724" x2="29.9175" y2="26.2041" width="0.2032" layer="1"/>
 <wire x1="29.9175" y1="26.2041" x2="20.3659" y2="26.2041" width="0.2032" layer="1"/>
 <wire x1="20.3659" y1="26.2041" x2="19.34" y2="27.23" width="0.2032" layer="1"/>
@@
 <via x="57.0037" y="35.3496" extent="1-16" drill="0.3048" diameter="0.6096"/>
 <via x="60.5619" y="24.4583" extent="1-16" drill="0.3048" diameter="0.6096"/>
-<wire x1="55.0467" y1="35.2535" x2="55.0467" y2="36.9215" width="0.2032" layer="1"/>
+<wire x1="55.0467" y1="35.2535" x2="55.0467" y2="36.4215" width="0.2032" layer="1"/>
 <wire x1="56.0257" y1="35.2457" x2="55.0545" y2="35.2457" width="0.2032" layer="1"/>
 <wire x1="55.0545" y1="35.2457" x2="55.0467" y2="35.2535" width="0.2032" layer="1"/>

Commit message: PCB/sch small changes. 19.2Mhz fix additional transistor PSU resistor fixes
Connections:
- removed net N$26: U$4.3, U1.11, U2.11
- removed net N$5: U1.1
- net N$7: now also U$4.3, U1.1, U1.11, U2.11
Routing:
- net N$7: track 0.00 -> 11.5 mm, vias 0 -> 1
- net N$26: track 11.5 -> 0.00 mm, vias 1 -> 0
Changed lines of the file:
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@@
 <grid distance="0.25" unitdist="mm" unit="mm" style="lines" multiple="1" display="yes" altdistance="0.003125" altunitdist="mic" altunit="mm"/>
 <layers>
-<layer number="1" name="Top" color="4" fill="1" visible="no" active="yes"/>
+<layer number="1" name="Top" color="4" fill="1" visible="yes" active="yes"/>
 <layer number="2" name="Route2" color="21" fill="1" visible="no" active="yes"/>
 <layer number="3" name="Route3" color="4" fill="3" visible="no" active="no"/>
@@
 <layer number="14" name="Route14" color="1" fill="6" visible="no" active="no"/>
 <layer number="15" name="Route15" color="16" fill="1" visible="no" active="yes"/>
-<layer number="16" name="Bottom" color="9" fill="1" visible="yes" active="yes"/>
+<layer number="16" name="Bottom" color="9" fill="1" visible="no" active="yes"/>
 <layer number="17" name="Pads" color="2" fill="1" visible="yes" active="yes"/>
 <layer number="18" name="Vias" color="2" fill="1" visible="yes" active="yes"/>
@@
 <via x="6.97933125" y="5.4862" extent="1-16" drill="0.6" diameter="0.6096"/>
 <via x="24.138159375" y="11.41869375" extent="1-16" drill="0.3048" diameter="0.6096"/>
-<wire x1="25.138159375" y1="11.41869375" x2="25.138159375" y2="11.41869375" width="0" layer="19" extent="1-16"/>
 <via x="28.638159375" y="10.66869375" extent="1-16" drill="0.3048" diameter="0.6096"/>
 <via x="28.638159375" y="9.66869375" extent="1-16" drill="0.3048" diameter="0.6096"/>
@@
 <via x="21" y="54.25" extent="1-16" drill="0.9" diameter="0.6096"/>
 </signal>
-<signal name="N$5">
-<contactref element="U1" pad="1"/>
-</signal>
 <signal name="N$7">
 <contactref element="U2" pad="1"/>
-</signal>
-<signal name="N$26">
+<contactref element="U1" pad="1"/>
 <contactref element="U1" pad="11"/>
 <contactref element="U2" pad="11"/>
@@
 <wire x1="56.878" y1="18.9608" x2="56.31" y2="18.3928" width="0.2032" layer="16"/>
 <via x="56.31" y="18.3928" extent="1-16" drill="0.3048" diameter="0.6096"/>
+<wire x1="58.6904" y1="19.7206" x2="59.9986" y2="23.1012" width="0" layer="19" extent="1-16"/>
+<wire x1="55.8446" y1="23.0989" x2="57.1528" y2="19.7229" width="0" layer="19" extent="1-16"/>
 </signal>
 <signal name="LX">
@@
 </signal>
 </signals>
-<errors>
-</errors>
 </board>
 </drawing>
